File: Electronics/Project Moonlight Motherboard/Project Moonlight Motherboard.kicad_pcb (KiCad board)
At the start: 4 copper layers, 113.4 x 56 mm, 45 parts, among them M1 AO3400A, M2 AO3400A, M3 AO3400A, U2 TMC2209_SILENTSTEPSTICK, U3 TMC2209_SILENTSTEPSTICK, U4 TMC2209_SILENTSTEPSTICK, U5 TMC2209_SILENTSTEPSTICK

Commit message: routed all new items
Parts:
- added D1: WS2812, LED_SMD:LED_WS2812_PLCC6_5.0x5.0mm_P1.6mm, F.Cu at (197.0, 108.1)
- added D2: WS2812, LED_SMD:LED_WS2812_PLCC6_5.0x5.0mm_P1.6mm, F.Cu at (209.1, 118.8)
- added D3: WS2812, LED_SMD:LED_WS2812_PLCC6_5.0x5.0mm_P1.6mm, F.Cu at (209.1, 124.6)
- added J1: DX07S024JJ3R1300, DX07S024JJ3R1300:JAE_DX07S024JJ3R1300, F.Cu at (105.0, 100.0)
- added R8: RMCF0805JT5K10, RMCF0805JT5K10:RESC2012X65N, F.Cu at (102.9, 106.8)
- added R9: RMCF0805JT5K10, RMCF0805JT5K10:RESC2012X65N, F.Cu at (102.9, 93.2)
- added U1: AMS1117-3.3, Package_TO_SOT_SMD:SOT-223-3_TabPin2, F.Cu at (209.8, 94.8)
- added U6: LM2576HVS-5, Package_TO_SOT_SMD:TO-263-5_TabPin3, F.Cu at (206.9, 79.0)
- moved SCRN1 1.81 mm to (200.4, 98.8)
- moved PWR1 1.60 mm to (210.0, 106.9)
- moved REN1 1.38 mm to (196.2, 98.8)
Connections:
- MCU1 pad 9: unconnected-(MCU1-PC15-Pad9) -> NEOPIXEL_DIN
Routing:
- net +5V: track 0.00 -> 232.2 mm, vias 0 -> 6
- net USB_DP: track 0.00 -> 92.6 mm, vias 0 -> 6
- net USB_DM: track 0.00 -> 90.9 mm, vias 0 -> 4
- net Net-(D1-DOUT): track 0.00 -> 35.0 mm, vias 0 -> 2
- net VCC: track 250.8 -> 282.8 mm, vias 0 -> 1
- net GNDREF: track 128.9 -> 157.6 mm, vias 10 -> 17
- net NEOPIXEL_DIN: track 0.00 -> 28.5 mm, vias 0 -> 2
- net Net-(J1-CC1): track 0.00 -> 12.0 mm
- net Net-(D2-DOUT): track 0.00 -> 9.90 mm
- net Net-(J1-CC2): track 0.00 -> 7.49 mm
- net Net-(F1-Pad1): track 14.6 -> 17.1 mm
- net EN_FOR: track 29.1 -> 30.6 mm
- net +3V3: track 301.3 -> 299.7 mm
- net SCRN_SDA: track 36.2 -> 35.4 mm
- net SCRN_SCL: track 38.0 -> 37.2 mm
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