File: Electronics/Project Moonlight Motherboard/Project Moonlight Motherboard.kicad_sch (KiCad schematic)
At the start: 47 parts, among them J1 DX07S024JJ3R1300, M1 AO3400A, M2 AO3400A, M3 AO3400A, U1 LM2576S-3.3_NOPB, U2 TMC2209_SILENTSTEPSTICK, U3 TMC2209_SILENTSTEPSTICK, U4 TMC2209_SILENTSTEPSTICK, U5 TMC2209_SILENTSTEPSTICK

Commit message: generate BOM
Parts:
- R8, R9: value 5.1K -> RMCF0805JT5K10; footprint (none) -> RMCF0805JT5K10:RESC2012X65N

Commit message: i want to *die* - voltage reg stuff
id get some1 to doubel check this shit lmaoooo
Parts:
- removed U1: LM2576S-3.3_NOPB, LM2576S-3.3_NOPB:VREG_TPS79625KTTR, symbol LM2576S-3.3_NOPB:LM2576S-3.3_NOPB
- added C10: UWT1V221MNL1GS, UWT1V221MNL1GS, symbol UWT1V101MCL1GS:UWT1V101MCL1GS
- added C8: UWT1V101MCL1GS, UWT1V101MCL1GS:CAPAE830X1000N, symbol UWT1V101MCL1GS:UWT1V101MCL1GS
- added C9: UWT1V331MNL1GS, UWT1V331MNL1GS:CAPAE830X1000N, symbol UWT1V101MCL1GS:UWT1V101MCL1GS
- added U1: AMS1117-3.3, Package_TO_SOT_SMD:SOT-223-3_TabPin2, symbol Regulator_Linear:AMS1117-3.3
- added U6: LM2576HVS-5, Package_TO_SOT_SMD:TO-263-5_TabPin3, symbol Regulator_Switching:LM2576HVS-5
Connections:
- net +3V3: now also C10.1, U1.2 (VO)
- net +5V: now also C9.1, U6.2 (OUT), U6.4 (FB)
- net GNDREF: now also J1.B1 (GNDB), J1.B12 (GNDB), J1.S1 (SHIELD), J1.S2 (SHIELD), C10.2, C8.2, C9.2, U1.1 (GND), U6.3 (GND), U6.5 (~{ON}/OFF)
- net VCC: now also C8.1, U1.3 (VI), U6.1 (VIN)

Commit message: i am skibidi and i add voltage and usb
Connections:
- net +5V: now also U1.3 (VI)
- net USB_DM: now also J1.A7 (DA-), J1.B7 (DB-)
- net USB_DP: now also J1.A6 (DA+), J1.B6 (DB+)
- net VCC: no longer U1.3 (VI)

Commit message: rgb stuff
Parts:
- added D1, D2, D3: WS2812, LED_SMD:LED_WS2812_PLCC6_5.0x5.0mm_P1.6mm, symbol LED:WS2812
- added RGB: B3B-XH-A, B3B-XH-A:JST_B3B-XH-A, symbol B3B-XH-A:B3B-XH-A
Connections:
- net +5V: now also D1.3 (VCC), D1.5 (VDD), D2.3 (VCC), D2.5 (VDD), D3.3 (VCC), D3.5 (VDD), RGB.3
- net GNDREF: now also D1.6 (VSS), D2.6 (VSS), D3.6 (VSS), RGB.1
- net NEOPIXEL_DIN: now reaches MCU1.9 (PC15)
- net NEOPIXEL_DIN: now also D1.2 (DIN)
- new net: D1.1 (DOUT), D2.2 (DIN)
- new net: D2.1 (DOUT), D3.2 (DIN)
- new net NEOPIXEL_DOUT: D3.1 (DOUT), RGB.2

Commit message: routed all new items
Parts:
- renumbered RGB to RGB1
