File: Electronics/Motherboard/Motherboard.kicad_sch (KiCad schematic)
At the start: 55 parts, among them J1 DX07S024JJ3R1300, M1 AO3400A, M2 AO3400A, M3 AO3400A, U1 AMS1117-3.3, U2 TMC2209_SILENTSTEPSTICK, U3 TMC2209_SILENTSTEPSTICK, U4 TMC2209_SILENTSTEPSTICK, U5 TMC2209_SILENTSTEPSTICK, U6 LM2576HVS-5

Commit message: added capacitors and JST connector (except 331 because i don't have CAD)
Parts:
- C10: footprint UWT1V221MNL1GS -> UWT1V221MNL1GS:CAPAE1030X1080N_UWT1H221MNL1GS
- RGB1: footprint B3B-XH-A:JST_B3B-XH-A -> B3B-XH-A:JST_B3B-XH-A_LF__SN_
