File: Electronics/Motherboard/Motherboard.kicad_pcb (KiCad board)
At the start: 4 copper layers, 113.4 x 56 mm, 56 parts, among them J1 DX07S024JJ3R1300, M1 AO3400A, M2 AO3400A, M3 AO3400A, U1 AMS1117-3.3, U2 TMC2209_SILENTSTEPSTICK, U3 TMC2209_SILENTSTEPSTICK, U4 TMC2209_SILENTSTEPSTICK, U5 TMC2209_SILENTSTEPSTICK, U6 LM2576HVS-5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

Commit message: more routing
Routing:
- net +5V: track 66.0 -> 234.2 mm, vias 2 -> 11
- net GNDREF: track 452.3 -> 545.2 mm, vias 5 -> 7
- net USB_DP: track 1.32 -> 58.9 mm, vias 0 -> 2
- net USB_DM: track 2.24 -> 48.5 mm
- net Net-(D2-DOUT): track 0.00 -> 46.2 mm
- net +3V3: track 257.2 -> 299.0 mm, vias 2 -> 3
- net NEOPIXEL_DOUT: track 0.00 -> 4.92 mm
- net UART_RX: track 6.31 -> 6.36 mm, vias 0 -> 2

Commit message: MORE POWAAAAA
Routing:
- net VCC: track 237.8 -> 277.0 mm, vias 10 -> 16
- net GNDREF: track 545.2 -> 583.9 mm, vias 7 -> 8
- net Net-(HOTEND1-Pad01): track 3.81 -> 31.7 mm
- net Net-(J1-CC1): track 0.00 -> 11.8 mm, vias 0 -> 2
- net +5V: track 234.2 -> 241.8 mm
- net Net-(F1-Pad1): track 30.5 -> 28.6 mm
- net Net-(BED1-Pad01): track 21.6 -> 23.0 mm
- net USB_DP: track 58.9 -> 60.0 mm, vias 2 -> 3

Commit message: so i kinda added an extra thing for more IO uhhhhhhhh
Parts:
- moved DEBUG1 30.7 mm to (164.5, 89.3), turned to -90 degrees
Routing:
- net Net-(D1-DOUT): track 0.00 -> 66.8 mm, vias 0 -> 2
- net NEOPIXEL_DIN: track 0.00 -> 33.8 mm, vias 0 -> 2
- net GNDREF: track 583.9 -> 614.3 mm, vias 8 -> 9
- net +3V3: track 299.0 -> 323.6 mm, vias 3 -> 4
- net +5V: track 241.8 -> 247.2 mm

Commit message: final routing!!!!
Parts:
- added J2: Conn_02x10_Odd_Even, 2x10_tht:PinBox-2.54-02x10-THT, F.Cu at (194.9, 101.0)
- moved R4 1.51 mm to (193.0, 118.7)
Connections:
- U7 pad 15: unconnected-(U7-PF0-Pad15) -> PF0
- U7 pad 16: unconnected-(U7-PF1-Pad16) -> PF1
- U7 pad 17: unconnected-(U7-PF2-Pad17) -> PF2
- U7 pad 18: unconnected-(U7-PF3-Pad18) -> PF3
- U7 pad 19: unconnected-(U7-PF4-Pad19) -> PF4
- U7 pad 20: unconnected-(U7-PF5-Pad20) -> PF5
- U7 pad 4: unconnected-(U7-PE4-Pad4) -> PE4
- U7 pad 5: unconnected-(U7-PE5-Pad5) -> PE5
- U7 pad 85: unconnected-(U7-PD7-Pad85) -> (no net)
Routing:
- net DIR_M1: track 0.00 -> 93.3 mm, vias 0 -> 1
- net DIAG_M1: track 0.00 -> 93.1 mm, vias 0 -> 1
- net UART_RX: track 6.36 -> 99.3 mm
- net STEP_M1: track 0.00 -> 90.3 mm, vias 0 -> 1
- net GNDREF: track 614.3 -> 702.2 mm, vias 9 -> 11
- net +3V3: track 323.6 -> 400.3 mm, vias 4 -> 11
- net HOTEND: track 0.00 -> 71.6 mm, vias 0 -> 6
- net DIR_M3: track 0.00 -> 67.9 mm, vias 0 -> 2
- net STEP_M3: track 0.00 -> 63.7 mm, vias 0 -> 1
- net DIAG_M3: track 0.00 -> 52.4 mm, vias 0 -> 1
- net BED: track 0.00 -> 49.7 mm, vias 0 -> 2
- net DIR_M2: track 0.00 -> 46.8 mm, vias 0 -> 3
- net EN_FOR: track 0.00 -> 45.9 mm, vias 0 -> 1
- net EN_REV: track 0.00 -> 41.9 mm, vias 0 -> 1
- net STEP_M2: track 0.00 -> 41.5 mm, vias 0 -> 3
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- removed copper zone on In1.Cu, net GNDREF
