File: Electronics/Motherboard/Motherboard.kicad_pcb (KiCad board)
At the start: 4 copper layers, 113.4 x 56 mm, 57 parts, among them J1 DX07S024JJ3R1300, J2 Conn_02x10_Odd_Even, M1 AO3400A, M2 AO3400A, M3 AO3400A, U1 AMS1117-3.3, U2 TMC2209_SILENTSTEPSTICK, U3 TMC2209_SILENTSTEPSTICK, U4 TMC2209_SILENTSTEPSTICK, U5 TMC2209_SILENTSTEPSTICK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

Commit message: tryna make a 2layer versin of this so itd be cheaper, wish me luck lol
uart and driver wirint done
Connections:
- Q1 pad 1: GNDREF -> unconnected-(Q1-S-Pad1)
- Q1 pad 2: GNDREF -> unconnected-(Q1-S-Pad2)
- Q1 pad 3: GNDREF -> unconnected-(Q1-S-Pad3)
- Q2 pad 1: GNDREF -> unconnected-(Q2-S-Pad1)
- Q2 pad 2: GNDREF -> unconnected-(Q2-S-Pad2)
- Q2 pad 3: GNDREF -> unconnected-(Q2-S-Pad3)
- U7 pad 21: STEP_M1 -> unconnected-(U7-PC0-Pad21)
- U7 pad 22: DIR_M1 -> unconnected-(U7-PC1-Pad22)
- U7 pad 23: DIAG_M1 -> unconnected-(U7-PC2-Pad23)
- U7 pad 24: DIR_M2 -> unconnected-(U7-PC3-Pad24)
- U7 pad 62: unconnected-(U7-PD11-Pad62) -> DIR_M2
- U7 pad 65: unconnected-(U7-PD12-Pad65) -> DIAG_M1
- U7 pad 66: unconnected-(U7-PD13-Pad66) -> DIR_M1
- U7 pad 67: unconnected-(U7-PD14-Pad67) -> STEP_M1
- U7 pad 68: unconnected-(U7-PD15-Pad68) -> EN_M1
- U7 pad 75: unconnected-(U7-PA15-Pad75) -> NEOPIXEL_DIN
- U7 pad 85: (no net) -> unconnected-(U7-PD7-Pad85)
- U7 pad 9: NEOPIXEL_DIN -> unconnected-(U7-PC14-Pad9)
Routing:
- net GNDREF: track 702.2 -> 0.00 mm, vias 11 -> 0
- net +3V3: track 400.3 -> 0.00 mm, vias 11 -> 0
- net VCC: track 277.0 -> 0.00 mm, vias 15 -> 0
- net +5V: track 243.6 -> 0.00 mm, vias 10 -> 0
- net EN_M1: track 0.00 -> 70.6 mm, vias 0 -> 3
- net Net-(D1-DOUT): track 68.0 -> 0.00 mm, vias 2 -> 0
- net USB_DP: track 60.7 -> 0.00 mm, vias 3 -> 0
- net USB_DM: track 49.9 -> 0.00 mm
- net Net-(D2-DOUT): track 46.2 -> 0.00 mm
- net EN_FOR: track 45.9 -> 0.00 mm, vias 1 -> 0
- net EN_REV: track 41.9 -> 0.00 mm, vias 1 -> 0
- net ABL: track 38.0 -> 0.00 mm, vias 1 -> 0
- net EN_BTN: track 36.7 -> 0.00 mm, vias 1 -> 0
- net SCRN_SCL: track 31.7 -> 0.00 mm, vias 1 -> 0
- net Net-(HOTEND1-Pad01): track 31.7 -> 0.00 mm
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Other:
- copper layers 4 -> 2
