File: Electronics/Motherboard/motherboard_2layers.kicad_pcb (KiCad board)
At the start: 2 copper layers, 113.4 x 56 mm, 56 parts, among them J2 Conn_02x10_Odd_Even, M1 AO3400A, M2 AO3400A, M3 AO3400A, U1 AMS1117-3.3, U6 LM2576HVS-5, U8 STM32F405RGTx

Commit message: rahhh work
Parts:
- renumbered RGB1 to RGB
Connections:
- S1 pad 3: Net-(U2-M1B) -> Net-(S1-M1B)
- S1 pad 4: Net-(U2-M1A) -> Net-(S1-M1A)
- S1 pad 5: Net-(U2-M2A) -> Net-(S1-M2A)
- S1 pad 6: Net-(U2-M2B) -> Net-(S1-M2B)
- S2 pad 3: Net-(U4-M1B) -> Net-(S2-M1B)
- S2 pad 4: Net-(U4-M1A) -> Net-(S2-M1A)
- S2 pad 5: Net-(U4-M2A) -> Net-(S2-M2A)
- S2 pad 6: Net-(U4-M2B) -> Net-(S2-M2B)
- S3 pad 3: Net-(U3-M1B) -> Net-(S3-M1B)
- S3 pad 4: Net-(U3-M1A) -> Net-(S3-M1A)
- S3 pad 5: Net-(U3-M2A) -> Net-(S3-M2A)
- S3 pad 6: Net-(U3-M2B) -> Net-(S3-M2B)
- S4 pad 3: Net-(U5-M1B) -> Net-(S4-M1B)
- S4 pad 4: Net-(U5-M1A) -> Net-(S4-M1A)
- S4 pad 5: Net-(U5-M2A) -> Net-(S4-M2A)
- S4 pad 6: Net-(U5-M2B) -> Net-(S4-M2B)
Routing:
- net +5V: track 241.5 -> 228.4 mm, vias 14 -> 6
- net USB_DP: track 52.3 -> 41.9 mm, vias 3 -> 2
- net HOTEND: track 69.7 -> 75.4 mm, vias 2 -> 4
- net Net-(U4-M1B): track 5.32 -> 0.00 mm
- net Net-(S2-M1B): track 0.00 -> 5.32 mm
- net Net-(U4-M1A): track 5.31 -> 0.00 mm
- net Net-(S2-M1A): track 0.00 -> 5.31 mm
- net Net-(U4-M2B): track 5.29 -> 0.00 mm
- net Net-(S2-M2B): track 0.00 -> 5.29 mm
- net Net-(U4-M2A): track 5.29 -> 0.00 mm
- net Net-(S2-M2A): track 0.00 -> 5.29 mm
- net VCC: track 257.5 -> 252.3 mm, vias 10 -> 2
- net Net-(U5-M2B): track 5.15 -> 0.00 mm
- net Net-(U5-M1B): track 5.15 -> 0.00 mm
- net Net-(S4-M2B): track 0.00 -> 5.15 mm
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
Commit message: finito for now
Parts:
- renumbered ABL1 to ABL, MOTOR_E1 to MOTOR_E, MOTOR_X1 to MOTOR_X, MOTOR_Y1 to MOTOR_Y, MOTOR_Z1 to MOTOR_Z, Z_END1 to Z_END
Routing:
- net UART_RX: track 94.0 -> 87.1 mm, vias 7 -> 6
- net +5V: track 228.4 -> 223.8 mm, vias 6 -> 8
- net HOTEND: track 75.4 -> 71.8 mm, vias 4 -> 2
- net VCC: track 252.3 -> 250.3 mm, vias 2 -> 0
- net Net-(D1-DOUT): track 69.6 -> 71.5 mm
- net DIAG_M1: track 62.0 -> 61.1 mm, vias 7 -> 5
- net +3V3: track 257.7 -> 256.9 mm
- net NEOPIXEL_DIN: track 24.8 -> 24.0 mm
- net DIR_M1: track 81.0 -> 80.5 mm
- net GNDREF: track 0.00 -> 0.22 mm, vias 0 -> 91
- net DIR_M2: track 31.7 -> 31.9 mm, vias 1 -> 2
- net NEOPIXEL_DOUT: track 4.92 -> 4.99 mm, vias 0 -> 1
- net ABL: vias 0 -> 1
- added copper zone on B.Cu, net GNDREF

Commit message: just fixing up some routing and doing drc stuff
Routing:
- net Net-(D1-DOUT): track 71.5 -> 37.7 mm, vias 4 -> 1
- net GNDREF: track 0.22 -> 3.21 mm, vias 91 -> 93
- net +5V: track 223.8 -> 221.6 mm
- net NEOPIXEL_DIN: track 24.0 -> 25.5 mm
- net Z_END: track 31.2 -> 31.5 mm, vias 0 -> 2
- net ABL: track 37.5 -> 37.4 mm, vias 1 -> 3

Commit message: more clean up neneds to be done
Routing:
- net Net-(D1-DOUT): track 37.7 -> 65.5 mm, vias 1 -> 4
- net STEP_M2: track 41.5 -> 37.5 mm
- net +5V: track 221.6 -> 218.9 mm
- net DIAG_M3: track 51.8 -> 49.2 mm
- net DIR_M3: track 60.3 -> 58.7 mm
- net UART_RX: track 87.1 -> 88.4 mm
- net +3V3: track 257.3 -> 256.7 mm, vias 11 -> 8
- net T1: vias 0 -> 2

Commit message: almost done for now
Parts:
- moved Q1 0.16 mm to (117.1, 85.4)
Connections:
- Q1 pad 1: unconnected-(Q1-S-Pad1) -> GNDREF
- Q1 pad 2: unconnected-(Q1-S-Pad2) -> GNDREF
- Q1 pad 3: unconnected-(Q1-S-Pad3) -> GNDREF
- Q2 pad 1: unconnected-(Q2-S-Pad1) -> GNDREF
- Q2 pad 2: unconnected-(Q2-S-Pad2) -> GNDREF
- Q2 pad 3: unconnected-(Q2-S-Pad3) -> GNDREF
Routing:
- net Net-(HOTEND1-Pad01): track 34.4 -> 0.00 mm
- net Net-(D1-DOUT): track 65.5 -> 61.7 mm
- net GNDREF: track 2.98 -> 4.23 mm, vias 93 -> 103
- net PB13: track 15.0 -> 14.4 mm
- net PB14: track 11.7 -> 11.2 mm
- net PB15: track 14.4 -> 13.8 mm
- net UART_RX: track 88.4 -> 87.9 mm
- net DIR_M4: track 13.3 -> 12.8 mm
- added copper zone on B.Cu, net Net-(BED1-Pad01)

Commit message: okay im actually done now
Routing:
- net VCC: track 250.3 -> 276.5 mm
- net GNDREF: vias 103 -> 139
- added copper zone on F.Cu, net Net-(HOTEND1-Pad01)
- removed copper zone on B.Cu, net Net-(BED1-Pad01)
