File: Electronics/Motherboard/motherboard_2layers.kicad_sch (KiCad schematic)
At the start: 54 parts, among them J2 Conn_02x10_Odd_Even, M1 AO3400A, M2 AO3400A, M3 AO3400A, U1 AMS1117-3.3, U6 LM2576HVS-5, U8 STM32F405RGTx

Commit message: added models and fixed screen header footprint
Parts:
- J2: footprint 2x10_tht:PinBox-2.54-02x10-THT -> Connector_PinHeader_2.54mm:PinHeader_2x10_P2.54mm_Vertical
Changed lines of the file:
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@@
 	)
 	(junction
-		(at 215.9 220.98)
-		(diameter 0)
-		(color 0 0 0 0)
-	)
-	(junction
 		(at 186.69 102.87)
 		(diameter 0)
@@
 	)
 	(junction
-		(at 215.9 218.44)
-		(diameter 0)
-		(color 0 0 0 0)
-	)
-	(junction
 		(at 375.92 35.56)
 		(diameter 0)
@@
 	)
 	(junction
-		(at 203.2 220.98)
-		(diameter 0)
-		(color 0 0 0 0)
-	)
-	(junction
-		(at 203.2 218.44)
+		(at 284.48 34.29)
 		(diameter 0)
 		(color 0 0 0 0)
 	)
 	(junction
-		(at 284.48 34.29)
+		(at 64.77 76.2)
 		(diameter 0)
 		(color 0 0 0 0)
 	)
 	(junction
-		(at 64.77 76.2)
+		(at 215.9 218.44)
 		(diameter 0)
 		(color 0 0 0 0)
@@
 	)
 	(junction
+		(at 203.2 218.44)
+		(diameter 0)
+		(color 0 0 0 0)
+	)
+	(junction
 		(at 283.21 118.11)
 		(diameter 0)
@@
 	)
 	(junction
+		(at 215.9 220.98)
+		(diameter 0)
+		(color 0 0 0 0)
+	)
+	(junction
 		(at 349.25 232.41)
 		(diameter 0)
@@
 		(color 0 0 0 0)
 	)
+	(junction
+		(at 203.2 220.98)
+		(diameter 0)
+		(color 0 0 0 0)
+	)
 	(wire
 		(pts
@@
 	(wire
 		(pts
+			(xy 215.9 220.98) (xy 215.9 226.06)
+		)
+		(stroke
+			(width 0)
+			(type default)
+		)
+	)
+	(wire
+		(pts
 			(xy 281.94 67.31) (xy 283.21 67.31)
 		)
@@
 	(wire
 		(pts
-			(xy 203.2 220.98) (xy 203.2 226.06)
-		)
-		(stroke
-			(width 0)
-			(type default)
-		)
-	)
-	(wire
-		(pts
 			(xy 157.48 264.16) (xy 154.94 264.16)
 		)
@@
 	(wire
 		(pts
+			(xy 203.2 218.44) (xy 203.2 220.98)
+		)
+		(stroke
+			(width 0)
+			(type default)
+		)
+	)
+	(wire
+		(pts
 			(xy 283.21 41.91) (xy 281.94 41.91)
 		)
@@
 	(wire
 		(pts
+			(xy 203.2 220.98) (xy 203.2 226.06)
+		)
+		(stroke
+			(width 0)
+			(type default)
+		)
+	)
+	(wire
+		(pts
 			(xy 210.82 139.7) (xy 210.82 142.24)
 		)
@@
 	(wire
 		(pts
-			(xy 215.9 218.44) (xy 215.9 220.98)
-		)
-		(stroke
-			(width 0)
-			(type default)
-		)
-	)
-	(wire
-		(pts
 			(xy 373.38 68.58) (xy 375.92 68.58)
 		)
@@
 	(wire
 		(pts
-			(xy 203.2 218.44) (xy 203.2 220.98)
+			(xy 203.2 215.9) (xy 203.2 218.44)
 		)
 		(stroke
@@
 	(wire
 		(pts
-			(xy 215.9 220.98) (xy 215.9 226.06)
+			(xy 199.39 92.71) (xy 205.74 92.71)
 		)
 		(stroke
@@
 	(wire
 		(pts
-			(xy 199.39 92.71) (xy 205.74 92.71)
+			(xy 215.9 218.44) (xy 215.9 220.98)
 		)
 		(stroke
@@
 		)
 	)
-	(wire
-		(pts
-			(xy 203.2 215.9) (xy 203.2 218.44)
-		)
-		(stroke
-			(width 0)
-			(type default)
-		)
-	)
 	(rectangle
 		(start 86.995 232.41)
@@
 	)
 	(symbol
+		(lib_id "Connector_Generic:Conn_02x10_Odd_Even")
+		(at 208.28 208.28 0)
+		(unit 1)
+		(exclude_from_sim no)
+		(in_bom yes)
+		(on_board yes)
+		(dnp no)
+		(fields_autoplaced yes)
+		(property "Reference" "J2"
+			(at 209.55 191.77 0)
+			(effects
+				(font
+					(size 1.27 1.27)
+				)
+			)
+		)
+		(property "Value" "Conn_02x10_Odd_Even"
+			(at 209.55 194.31 0)
+			(effects
+				(font
+					(size 1.27 1.27)
+				)
+			)
+		)
+		(property "Footprint" "Connector_PinHeader_2.54mm:PinHeader_2x10_P2.54mm_Vertical"
+			(at 208.28 208.28 0)
+			(effects
+				(font
+					(size 1.27 1.27)
+				)
+				(hide yes)
+			)
+		)
+		(property "Datasheet" "~"
+			(at 208.28 208.28 0)
+			(effects
+				(font
+					(size 1.27 1.27)
+				)
+				(hide yes)
+			)
+		)
+		(property "Description" "Generic connector, double row, 02x10, odd/even pin numbering scheme (row 1 odd numbers, row 2 even numbers), script generated (kicad-library-utils/schlib/autogen/connector/)"
+			(at 208.28 208.28 0)
+			(effects
+				(font
+					(size 1.27 1.27)
+				)
+				(hide yes)
+			)
+		)
+		(pin "14"
+		)
+		(pin "8"
+		)
+		(pin "17"
+		)
+		(pin "7"
+		)
+		(pin "9"
+		)
+		(pin "18"
+		)
+		(pin "12"
+		)
+		(pin "19"
+		)
+		(pin "6"
+		)
+		(pin "3"
+		)
+		(pin "11"
+		)
+		(pin "15"
+		)
+		(pin "4"
+		)
+		(pin "1"
+		)
+		(pin "5"
+		)
+		(pin "20"
+		)
+		(pin "13"
+		)
+		(pin "16"
+		)
+		(pin "10"
+		)
+		(pin "2"
+		)
+		(instances
+			(project ""
+				(path "/9290e430-09f5-4a3f-8744-4071dceedc2e"
+					(reference "J2")
+					(unit 1)
+				)
+			)
+		)
+	)
+	(symbol
 		(lib_id "power:+5V")
 		(at 203.2 200.66 90)
@@
 					(unit 1)
 				)
-			)
-		)
-	)
-	(symbol
-		(lib_id "Connector_Generic:Conn_02x10_Odd_Even")
-		(at 208.28 208.28 0)
-		(unit 1)
-		(exclude_from_sim no)
-		(in_bom yes)
-		(on_board yes)
-		(dnp no)
-		(property "Reference" "J2"
-			(at 209.55 195.326 0)
-			(effects
-				(font
-					(size 1.27 1.27)
-				)
-			)
-		)
-		(property "Value" "Conn_02x10_Odd_Even"
-			(at 209.55 194.056 0)
-			(effects
-				(font
-					(size 1.27 1.27)
-				)
-				(hide yes)
-			)
-		)
-		(property "Footprint" "2x10_tht:PinBox-2.54-02x10-THT"
-			(at 208.28 208.28 0)
-			(effects
-				(font
-					(size 1.27 1.27)
-				)
-				(hide yes)
-			)
-		)
-		(property "Datasheet" "~"
-			(at 208.28 208.28 0)
-			(effects
-				(font
-					(size 1.27 1.27)
-				)
-				(hide yes)
-			)
-		)
-		(property "Description" "Generic connector, double row, 02x10, odd/even pin numbering scheme (row 1 odd numbers, row 2 even numbers), script generated (kicad-library-utils/schlib/autogen/connector/)"
-			(at 208.28 208.28 0)
-			(effects
-				(font
-					(size 1.27 1.27)
-				)
-				(hide yes)
-			)
-		)
-		(pin "10"
-		)
-		(pin "6"
-		)
-		(pin "17"
-		)
-		(pin "3"
-		)
-		(pin "13"
-		)
-		(pin "4"
-		)
-		(pin "1"
-		)
-		(pin "14"
-		)
-		(pin "16"
-		)
-		(pin "7"
-		)
-		(pin "20"
-		)
-		(pin "11"
-		)
-		(pin "12"
-		)
-		(pin "19"
-		)
-		(pin "9"
-		)
-		(pin "15"
-		)
-		(pin "18"
-		)
-		(pin "8"
-		)
-		(pin "5"
-		)
-		(pin "2"
-		)
-		(instances
-			(project ""
-				(path "/9290e430-09f5-4a3f-8744-4071dceedc2e"
-					(reference "J2")
-					(unit 1)
-				)
