File: Electronics/i2c screen/i2c screen.kicad_pcb (KiCad board)
At the start: 2 copper layers, 3 parts, among them J1 renc_con, J2 display_con, J3 display_in

Commit message: routing finito and placemnt aswell
Parts:
- added SW1: RotaryEncoder, Rotary_Encoder:RotaryEncoder_Bourns_Vertical_PEC12R-3x17F-Sxxxx, F.Cu at (180.5, 135.8)
- J3: footprint Connector_PinHeader_2.54mm:PinHeader_1x04_P2.54mm_Vertical -> ledscreen:128x64OLED
- moved J1 39.4 mm to (132.5, 131.0)
- moved J3 33.8 mm to (156.7, 127.7)
- moved J2 30.8 mm to (132.5, 119.0)
Routing:
- net EN_BTN: track 0.00 -> 55.2 mm
- net EN_REV: track 0.00 -> 51.3 mm
- net EN_FOR: track 0.00 -> 48.9 mm
- net Net-(J2-sda): track 0.00 -> 32.2 mm
- net Net-(J2-scl): track 0.00 -> 28.6 mm
- net Net-(J2-3v3): track 0.00 -> 25.0 mm
- net Net-(J2-gnd): track 0.00 -> 21.4 mm
- added copper zone on B.Cu, net GNDREF
- added copper zone on F.Cu, net GNDREF
Other:
- board outline added: 65 x 29 mm

Commit message: artwork!
Parts:
- added G***: LOGO, LOGO, F.Cu at (175.5, 139.5)
- added G***: LOGO, LOGO, F.Cu at (189.5, 139.5)
- added G***: LOGO, LOGO, F.Cu at (139.5, 139.0)
- added G***: LOGO, LOGO, F.Cu at (185.5, 117.0)
- added G***: LOGO, LOGO, B.Cu at (160.5, 128.0)
- SW1: value RotaryEncoder -> Encoder
Routing:
- net GNDREF: track 0.00 -> 69.5 mm
- removed copper zone on B.Cu, net GNDREF
- removed copper zone on F.Cu, net GNDREF
Other:
- board text added: "PCB by @awdev and @blaze"
- board text added: "it's been a while in the working, thanks to everyone on the forge team for your help and thank YOU for making it possible!"
